Commit message: update: launch file, packages file and paramater files are crated for ros1 support

File: urdf files/robot_arm_urdf/urdf/robot_arm_urdf.urdf (robot description, URDF)
Before this commit: robot robot_arm_urdf, 8 links, 7 joints
Links:
- added link world
Joints:
- added joint base_joint: type fixed, parent world, child base_link, origin xyz=0.0 0.0 0.17 rpy=0 0 0
- joint joint_4: limit lower=0 upper=-3.142 effort=200 velocity=3 -> lower=-3.142 upper=0 effort=200 velocity=3
